Commit message: Etape 2 new file:   description/gazebo_control.xacro modified:   description/robot.urdf.xacro modified:   description/robot_core.xacro new file:   launch/launch_sim.launch.py

File: description/robot.urdf.xacro (robot description, xacro)
@@ -2,3 +2,4 @@
 <robot xmlns:xacro="http://www.ros.org/wiki/xacro"  name="robot">
     <xacro:include filename="robot_core.xacro"/>
+     <xacro:include filename="gazebo_control.xacro"/>
 </robot>

File: description/robot_core.xacro (robot description, xacro)
@@ -6,6 +6,12 @@
   </link>
   <!--Chassis-->
+  <joint name="chassis_joint" type="fixed">
+    <parent link="base_link"/>
+    <child link="chassis"/>
+    <origin xyz="-0.06 0 0"/>
+  </joint>
   <link name="chassis">
     <visual>
+      <origin xyz="0.078 0 0.02"/>
       <geometry>
         <box size="0.18 0.12 0.05"/>
@@ -14,17 +20,16 @@
     </visual>
     <collision>
+      <origin xyz="0.078 0 0.02"/>
       <geometry>
         <box size="0.18 0.12 0.05"/>
       </geometry>
-      <material name="white"/>
     </collision>
     <xacro:inertial_box mass="0.15" x="0.18" y="0.12" z="0.05">
-        <origin xyz="0 0 0" rpy="0 0 0"/>
+        <origin xyz="0.078 0 0.02" rpy="0 0 0"/>
     </xacro:inertial_box>
   </link>
-  <joint name="chassis_joint" type="fixed">
-    <parent link="base_link"/>
-    <child link="chassis"/>
-  </joint>
+  <gazebo reference="chassis">
+    <material>Gazebo/White</material>
+  </gazebo>
   <!--Materials-->
   <material name="blue">
@@ -38,4 +43,10 @@
   </material>
   <!--Front wheel right-->
+  <joint name="front_wheel_right_joint" type="continuous">
+    <parent link="base_link"/>
+    <child link="front_wheel_right"/>
+    <origin xyz="0.08 -0.07 0" rpy="${pi/2} 0 0"/>
+    <axis xyz="0 0 -1"/>
+  </joint>
   <link name="front_wheel_right">
     <visual>
@@ -49,5 +60,4 @@
         <cylinder length="0.02" radius="0.02"/>
       </geometry>
-      <material name="blue"/>
     </collision>
     <xacro:inertial_cylinder mass="0.05" length="0.02" radius="0.02">
@@ -55,10 +65,7 @@
     </xacro:inertial_cylinder>
   </link>
-  <joint name="front_wheel_right_joint" type="continuous">
-    <parent link="base_link"/>
-    <child link="front_wheel_right"/>
-    <origin xyz="0.08 -0.075 -0.02" rpy="${pi/2} 0 0"/>
-    <axis xyz="0 0 -1"/>
-  </joint>
+  <gazebo reference="front_wheel_right">
+    <material>Gazebo/Black</material>
+  </gazebo>
   <!--Front wheel left-->
   <link name="front_wheel_left">
@@ -73,5 +80,4 @@
         <cylinder length="0.02" radius="0.02"/>
       </geometry>
-      <material name="blue"/>
     </collision>
     <xacro:inertial_cylinder mass="0.05" length="0.02" radius="0.02">
@@ -79,8 +85,11 @@
     </xacro:inertial_cylinder>
   </link>
+  <gazebo reference="front_wheel_left">
+    <material>Gazebo/Black</material>
+  </gazebo>
   <joint name="front_wheel_left_joint" type="continuous">
     <parent link="base_link"/>
     <child link="front_wheel_left"/>
-    <origin xyz="0.08 0.075 -0.02" rpy="-${pi/2} 0 0"/>
+    <origin xyz="0.08 0.07 0" rpy="-${pi/2} 0 0"/>
     <axis xyz="0 0 1"/>
   </joint>
@@ -97,5 +106,4 @@
         <cylinder length="0.02" radius="0.02"/>
       </geometry>
-      <material name="blue"/>
     </collision>
     <xacro:inertial_cylinder mass="0.05" length="0.02" radius="0.02">
@@ -103,11 +111,22 @@
     </xacro:inertial_cylinder>
   </link>
+  <gazebo reference="rear_wheel_right">
+    <material>Gazebo/Black</material>
+    <mu1 value="0.001"/>
+    <mu2 value="0.001"/>
+  </gazebo>
   <joint name="rear_wheel_right_joint" type="continuous">
     <parent link="base_link"/>
     <child link="rear_wheel_right"/>
-    <origin xyz="-0.08 -0.075 -0.02" rpy="${pi/2} 0 0"/>
+    <origin xyz="-0.04 -0.07 0" rpy="${pi/2} 0 0"/>
     <axis xyz="0 0 -1"/>
   </joint>
   <!--Rear wheel left-->
+  <joint name="rear_wheel_left_joint" type="continuous">
+    <parent link="base_link"/>
+    <child link="rear_wheel_left"/>
+    <origin xyz="-0.04 0.07 0" rpy="-${pi/2} 0 0"/>
+    <axis xyz="0 0 1"/>
+  </joint>
   <link name="rear_wheel_left">
     <visual>
@@ -121,5 +140,4 @@
         <cylinder length="0.02" radius="0.02"/>
       </geometry>
-      <material name="blue"/>
     </collision>
     <xacro:inertial_cylinder mass="0.05" length="0.02" radius="0.02">
@@ -127,9 +145,8 @@
     </xacro:inertial_cylinder>
   </link>
-  <joint name="rear_wheel_left_joint" type="continuous">
-    <parent link="base_link"/>
-    <child link="rear_wheel_left"/>
-    <origin xyz="-0.08 0.075 -0.02" rpy="-${pi/2} 0 0"/>
-    <axis xyz="0 0 1"/>
-  </joint>
+  <gazebo reference="rear_wheel_left">
+    <material>Gazebo/Black</material>
+    <mu1 value="0.001"/>
+    <mu2 value="0.001"/>
+  </gazebo>
 </robot>
